File: GP Layout/MOTOR_DRIVER_old.brd (EAGLE design)
At the start: 160 x 100 mm, 32 parts, among them U1 CSD18502KCS_KCS_3, U2 CSD18502KCS_KCS_3, U3 MIC4604YM, U4 CSD18502KCS_KCS_3, U5 CSD18502KCS_KCS_3, U6 MIC4604YM, U7 ATMEGA328P_TQFP, Y1 16MHz

Commit message: Updated all schematic sheets
Parts:
- removed D3, D4: BYV32, diode:TO220ABS
- removed S1: SWS006, smd-special:SMS-006
- C7: value 10uF -> (none)
- moved JP3 146.6 mm to (77.5, 17.8), flipped to the bottom
- moved R1 140.6 mm to (74.9, 25.4), turned to 90 degrees
- moved JP4 139.3 mm to (78.7, 22.9), turned to 270 degrees
- moved JP2 127.9 mm to (78.7, 38.1), flipped to the bottom, turned to 90 degrees
- moved JP5 114.2 mm to (86.4, 29.2), turned to 90 degrees
- moved U5 114.0 mm to (66.0, 39.4), turned to 90 degrees
- moved D2 112.1 mm to (49.5, 36.8), turned to 270 degrees
- moved U4 106.6 mm to (72.4, 39.4), turned to 90 degrees
- moved Y1 104.9 mm to (57.1, 26.7)
- moved U6 104.6 mm to (39.4, 26.7), turned to 270 degrees
- moved D1 102.0 mm to (50.8, 36.8), turned to 90 degrees
- moved U7 101.9 mm to (82.5, 8.89)
- moved C4 97.9 mm to (39.4, 34.3)
- moved C5 94.4 mm to (66.0, 26.7), turned to 90 degrees
- moved C7 92.4 mm to (71.1, 25.4), turned to 90 degrees
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Connections:
- removed net 5V_TEENSY: S1.6, U$1.VIN
- removed net 7_4V1: D4.A1, D4.A2
- removed net N$14: D4.C
- removed net N$17: LSP1.MP
- removed net REC_MOTOR: JP5.20, U$1.15/A1
- removed net REC_SERVO: U$1.18/A4/SDA
- removed net SW1: S1.1, U$1.24
- removed net SW2: S1.2, U$1.25
- removed net SW3: S1.3, U$1.26
- removed net SW4: S1.4, U$1.27
- removed net SW5: S1.5, U$1.28
- new net M2_GPIO1: JP5.10, U$1.19/A5/SCL
- new net M2_GPIO2: JP5.12, U$1.18/A4/SDA
- new net M2_GPIO3: JP5.14, U$1.A22/DAC1
- new net M2_GPIO4: JP5.16, U$1.21/DAC0
- new net M2_GPIO5: JP5.18, U$1.39/A20
- new net RECEIVER: JP5.20, U$1.5
- new net SWITCHES: U$1.33/A14, U$1.34/A15, U$1.35/A16, U$1.36/A17
- net 5V: now also U$1.VIN; no longer S1.7
- net 7_4V: now also LSP1.MP, U$2.3; no longer D3.A1, D3.A2
- net BLT_RX: now also U$1.0/RX; no longer U$1.7
- net BLT_TX: now also U$1.1/TX; no longer U$1.8
- net GND: no longer S1.10, S1.11, S1.12, S1.8, S1.9
- net HALL: now also U7.13; no longer U7.32
- net M1_GPIO3: now also U7.32; no longer U7.13
- net N$5: no longer D3.C
- net SERVO: now also U$1.16/A2; no longer U$1.20/A6
Routing:
- net GND: track 0.00 -> 234.4 mm, vias 0 -> 2
- net 7_4V: track 0.00 -> 140.7 mm, vias 0 -> 3
- net CAMERA_CLK: track 0.00 -> 139.6 mm, vias 0 -> 3
- net 5V: track 0.00 -> 134.9 mm, vias 0 -> 1
- net 3_3V: track 0.00 -> 94.2 mm, vias 0 -> 1
- net N$8: track 0.00 -> 89.9 mm
- net RECEIVER: track 0.00 -> 88.9 mm, vias 0 -> 1
- net N$1: track 0.00 -> 73.2 mm
- net M2_GPIO1: track 0.00 -> 70.1 mm, vias 0 -> 2
- net SERVO: track 0.00 -> 60.8 mm
- net M2_GPIO2: track 0.00 -> 58.1 mm, vias 0 -> 1
- net HI: track 0.00 -> 51.7 mm
- net M2_GPIO5: track 0.00 -> 47.3 mm, vias 0 -> 2
- net M2_GPIO3: track 0.00 -> 47.2 mm, vias 0 -> 2
- net HALL: track 0.00 -> 45.6 mm, vias 0 -> 2
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Other:
- board size 160 x 100 mm -> 91.4 x 45.4 mm
