File: GP Layout/MOTOR_DRIVER.brd (EAGLE design)
At the start: 91.4 x 97.5 mm, 46 parts, among them U3 MIC4604YM, U6 MIC4604YM, U7 ATMEGA328P_TQFP, Y1 16MHz

Commit message: fixed LI2 and HI2 errors
Connections:
- removed net HI_TOP: U6.6
- removed net LI_TOP: U6.5
- net HI2_TOP: now also U6.6
- net LI2_TOP: now also U6.5
Changed lines of the file:
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@@
 <wire x1="10.16" y1="24.13" x2="59.2074" y2="16.91" width="0" layer="19" extent="1-1"/>
-</signal>
-<signal name="LI_TOP">
-<contactref element="U6" pad="5"/>
-</signal>
-<signal name="HI_TOP">
-<contactref element="U6" pad="6"/>
 </signal>
 <signal name="GND_TOP">
@@
 <signal name="HI2_TOP">
 <contactref element="SV6" pad="3"/>
+<contactref element="U6" pad="6"/>
+<wire x1="15.24" y1="55.88" x2="31.115" y2="72.2757" width="0" layer="19" extent="16-16"/>
 </signal>
 <signal name="LI2_TOP">
 <contactref element="SV6" pad="4"/>
+<contactref element="U6" pad="5"/>
+<wire x1="17.78" y1="55.88" x2="32.385" y2="72.2757" width="0" layer="19" extent="16-16"/>
 </signal>
 </signals>
