File: GP Layout/MOTOR_DRIVER.brd (EAGLE design)
At the start: 91.4 x 97.5 mm, 46 parts, among them U3 MIC4604YM, U6 MIC4604YM, U7 ATMEGA328P_TQFP, Y1 16MHz

Commit message: added backup pins on Teensy for camera and HES
Connections:
- removed net N$36: SV4.7
- removed net N$37: SV4.6
- removed net N$38: SV4.5
- removed net N$39: SV4.4
- removed net N$40: SV4.3
- removed net N$41: SV4.2
- removed net N$42: SV4.1
- new net CAMERA_A0_BACKUP: SV4.1, U$1.31/A12
- new net CAMERA_CL_BACKUP: SV4.2, U$1.30
- new net CAMERA_SI_BACKUP: SV4.3, U$1.29
- new net HALL1_BACKUP: SV4.6, U$1.39/A20
- new net HALL2_BACKUP: SV4.7, U$1.38/A19
- net 3_3V: now also SV4.5
- net GND: now also SV4.4
Changed lines of the file:
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@@
 <contactref element="R2" pad="1"/>
 <contactref element="SV1" pad="10"/>
+<contactref element="SV4" pad="4"/>
 <wire x1="-29.464" y1="24.892" x2="-86.498" y2="-29.21" width="0" layer="19" extent="1-1"/>
 <wire x1="-37.084" y1="38.1" x2="-29.464" y2="24.892" width="0" layer="19" extent="1-1"/>
@@
 <wire x1="79.3242" y1="12.7" x2="79.3242" y2="15.24" width="0" layer="19" extent="1-1"/>
 <wire x1="79.3242" y1="10.16" x2="79.3242" y2="12.7" width="0" layer="19" extent="1-1"/>
+<wire x1="66.04" y1="3.81" x2="67.7926" y2="16.91" width="0" layer="19" extent="1-1"/>
 <wire x1="58.42" y1="38.1" x2="53.34" y2="21.59" width="0" layer="19" extent="1-1"/>
 <wire x1="63.5" y1="40.64" x2="58.42" y2="38.1" width="0" layer="19" extent="1-1"/>
@@
 <contactref element="U$1" pad="3V3_LO"/>
 <contactref element="SV3" pad="9"/>
+<contactref element="SV4" pad="5"/>
+<wire x1="68.58" y1="3.81" x2="68.58" y2="40.64" width="0" layer="19" extent="1-1"/>
 <wire x1="15.24" y1="24.13" x2="68.58" y2="40.64" width="0" layer="19" extent="1-1"/>
 </signal>
@@
 <contactref element="SV4" pad="8"/>
 </signal>
-<signal name="N$36">
-<contactref element="SV4" pad="7"/>
-</signal>
-<signal name="N$37">
-<contactref element="SV4" pad="6"/>
-</signal>
-<signal name="N$38">
-<contactref element="SV4" pad="5"/>
-</signal>
-<signal name="N$39">
-<contactref element="SV4" pad="4"/>
-</signal>
-<signal name="N$40">
-<contactref element="SV4" pad="3"/>
-</signal>
-<signal name="N$41">
-<contactref element="SV4" pad="2"/>
-</signal>
-<signal name="N$42">
-<contactref element="SV4" pad="1"/>
-</signal>
 <signal name="N$20">
 <contactref element="SV3" pad="4"/>
@@
 <wire x1="17.78" y1="55.88" x2="32.385" y2="72.2757" width="0" layer="19" extent="16-16"/>
 </signal>
+<signal name="CAMERA_SI_BACKUP">
+<contactref element="U$1" pad="29"/>
+<contactref element="SV4" pad="3"/>
+<wire x1="63.5" y1="3.81" x2="60.96" y2="8.89" width="0" layer="19" extent="1-1"/>
+</signal>
+<signal name="CAMERA_CL_BACKUP">
+<contactref element="U$1" pad="30"/>
+<contactref element="SV4" pad="2"/>
+<wire x1="60.96" y1="3.81" x2="63.5" y2="8.89" width="0" layer="19" extent="1-1"/>
+</signal>
+<signal name="CAMERA_A0_BACKUP">
+<contactref element="U$1" pad="31/A12"/>
+<contactref element="SV4" pad="1"/>
+<wire x1="58.42" y1="3.81" x2="66.04" y2="8.89" width="0" layer="19" extent="1-1"/>
+</signal>
+<signal name="HALL1_BACKUP">
+<contactref element="U$1" pad="39/A20"/>
+<contactref element="SV4" pad="6"/>
+<wire x1="71.12" y1="3.81" x2="53.34" y2="24.13" width="0" layer="19" extent="1-1"/>
+</signal>
+<signal name="HALL2_BACKUP">
+<contactref element="U$1" pad="38/A19"/>
+<contactref element="SV4" pad="7"/>
+<wire x1="73.66" y1="3.81" x2="55.88" y2="24.13" width="0" layer="19" extent="1-1"/>
+</signal>
 </signals>

Commit message: t :wq # Explicit paths specified without -i or -o; assuming --only paths...
Parts:
- removed D1, D2: BYV32, diode:TO220ABS
- removed SV3: (no value), con-lsta:FE10-2
- removed SV4: (no value), con-lsta:FE10
- removed U$3: LM1086IT-5.0/NOPB, TI1086:T03B
- added BLUETOOTH: (no value), con-lsta:FE04-1
- added CAMERA, CAMERA_B: (no value), con-lsta:FE05-1
- added HALL1, HALL1_B, HALL2, HALL2_B, SERVO: (no value), con-lstb:MA03-1
- added REC: (no value), con-lstb:MA06-1
- added TXRX: (no value), con-lsta:FE02-1
- added VOLT_REG: LM1086TO220V, v-reg-3:TO220S
- moved U$6 137.5 mm to (149.6, 84.8)
- moved U$2 132.3 mm to (140.0, 85.3)
- moved R1 128.4 mm to (30.0, 33.6)
- moved R2 128.4 mm to (26.4, 33.6)
- moved R3 128.4 mm to (22.8, 33.6)
- moved R4 128.4 mm to (19.3, 33.6)
- moved U$4 102.1 mm to (118.6, 86.1)
- moved U$5 100.8 mm to (114.0, 86.6)
- moved LSP4 52.8 mm to (3.97, 71.9)
- moved LSP5 42.7 mm to (3.67, 66.5)
- moved C8 40.7 mm to (6.60, 37.8)
- moved S1 6.32 mm to (82.6, 10.3)
- moved U$1 5.44 mm to (32.7, 17.2)
- moved FUSE 5.22 mm to (-65.3, 64.9), turned to 270 degrees
- moved SV5 3.34 mm to (24.5, 94.3)
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Connections:
- removed net CAMERA_A0_BACKUP: SV4.1, U$1.31/A12
- removed net CAMERA_CLK: SV3.13, U7.12
- removed net CAMERA_CL_BACKUP: SV4.2, U$1.30
- removed net CAMERA_SI_BACKUP: SV4.3, U$1.29
- removed net HALL: SV3.16, U7.32
- removed net HALL1_BACKUP: SV4.6, U$1.39/A20
- removed net HALL2_BACKUP: SV4.7, U$1.38/A19
- removed net N$1: D1.A1, D1.A2, R3.1, R4.2
- removed net N$20: SV3.4
- removed net N$33: SV4.10
- removed net N$34: SV4.9
- removed net N$35: SV4.8
- new net CAMERA_A0_B: CAMERA_B.3, U$1.31/A12
- new net CAMERA_CL: CAMERA.4, U7.12
- new net CAMERA_CL_B: CAMERA_B.4, U$1.30
- new net CAMERA_SI_B: CAMERA_B.5, U$1.29
- new net HALL1: HALL1.3, U7.32
- new net HALL1_B: HALL1_B.3, U$1.39/A20
- new net HALL2: HALL2.3
- new net HALL2_B: HALL2_B.3, U$1.38/A19
- new net REC_EXTRA1: REC.5
- new net REC_EXTRA2: REC.6
- net 3_3V: now also BLUETOOTH.4, CAMERA.2, CAMERA_B.2, HALL1.1, HALL1_B.1, HALL2.1, HALL2_B.1; no longer SV3.9, SV4.5
- net 5V: now also REC.2, SERVO.2, VOLT_REG.2; no longer SV1.8, SV3.18, SV3.6, SV3.7, U$3.2
- net 7_4V: now also VOLT_REG.3; no longer U$3.3
- net BLT_RX: now also BLUETOOTH.1; no longer SV3.1
- net BLT_TX: now also BLUETOOTH.2; no longer SV3.3
- net CAMERA_A0: now also CAMERA.3; no longer SV3.17
- net CAMERA_SI: now also CAMERA.5; no longer SV3.15
- net EMF_SENSE_HIGH: now also R3.1, R4.2; no longer D1.C
- net EMF_SENSE_LOW: now also S1.5; no longer D2.C
- net GND: now also BLUETOOTH.3, CAMERA.1, CAMERA_B.1, HALL1.2, HALL1_B.2, HALL2.2, HALL2_B.2, REC.1, SERVO.1, VOLT_REG.1; no longer S1.8, SV3.11, SV3.12, SV3.14, SV3.2, SV3.5, SV4.4, U$3.1
- net MOTOR_HIGH_TOP: now also SV6.5
- net MOTOR_LOW: now also S1.8; no longer D2.A1, D2.A2
- net MOTOR_LOW_TOP: no longer SV6.5
- net REC_MOTOR: now also REC.3; no longer SV3.8
- net REC_SERVO: now also REC.4; no longer SV3.10
- net RX: now also TXRX.1; no longer SV3.20
- net SERVO: now also SERVO.3; no longer SV1.9
- net SW5: no longer S1.5
- net TX: now also TXRX.2; no longer SV3.19
